File: miiMacRo.sch (KiCad schematic (older format))
At the start: 14 parts, among them SW1 SW_PUSH, SW10 SW_PUSH, SW11 SW_PUSH, SW12 Rotary_Encoder_Switch, SW2 SW_PUSH, SW3 SW_PUSH, SW4 SW_PUSH, SW5 SW_PUSH, SW6 SW_PUSH, SW7 SW_PUSH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

Commit message: first complete pcb
Parts:
- added H1, H2, H3, H4: MountingHole, kbd:M2_Hole_TH, symbol Mechanical:MountingHole
- SW1: value SW_PUSH -> 1; footprint Keebio-Parts:MX-Alps-Choc-1U-NoLED -> MX_Only:MXOnly-1U-NoLED
- SW10: value SW_PUSH -> 8; footprint Keebio-Parts:MX-Alps-Choc-1U-NoLED -> MX_Only:MXOnly-1U-NoLED
- SW11: value SW_PUSH -> 0; footprint Keebio-Parts:MX-Alps-Choc-1U-NoLED -> MX_Only:MXOnly-1U-NoLED
- SW12: value Rotary_Encoder_Switch -> ROTARY
- SW2: value SW_PUSH -> 5; footprint Keebio-Parts:MX-Alps-Choc-1U-NoLED -> MX_Only:MXOnly-1U-NoLED
- SW3: value SW_PUSH -> ENTER; footprint Keebio-Parts:MX-Alps-Choc-2U -> MX_Only:MXOnly-2U-ReversedStabilizers-NoLED
- SW4: value SW_PUSH -> 2; footprint Keebio-Parts:MX-Alps-Choc-1U-NoLED -> MX_Only:MXOnly-1U-NoLED
- SW5: value SW_PUSH -> 6; footprint Keebio-Parts:MX-Alps-Choc-1U-NoLED -> MX_Only:MXOnly-1U-NoLED
- SW6: value SW_PUSH -> 3; footprint Keebio-Parts:MX-Alps-Choc-1U-NoLED -> MX_Only:MXOnly-1U-NoLED
- SW7: value SW_PUSH -> 7; footprint Keebio-Parts:MX-Alps-Choc-1U-NoLED -> MX_Only:MXOnly-1U-NoLED
- SW8: value SW_PUSH -> 9; footprint Keebio-Parts:MX-Alps-Choc-1U-NoLED -> MX_Only:MXOnly-1U-NoLED
- SW9: value SW_PUSH -> 4; footprint Keebio-Parts:MX-Alps-Choc-1U-NoLED -> MX_Only:MXOnly-1U-NoLED
Connections:
- net +5V: now also U1.21 (VCC)
- net GND: now also SW12.S1; no longer SW12.S2
- net E6: now reaches SW1.2
- net E6: now also U1.10 (7/E6)
- net B4: now reaches U1.11 (8/B4)
- net B4: now also SW10.2
- net B5: now reaches U1.12 (9/B5)
- net B5: now also SW7.2
- net B6: now reaches U1.13 (B6/10)
- net B6: now also SW12.S2
- net B2: now reaches U1.14 (B2/16)
- net B2: now also SW5.2
- net B3: now reaches U1.15 (B3/14)
- net B3: now also SW2.2
- net B1: now reaches U1.16 (B1/15)
- net B1: now also SW11.2
- net F7: now reaches U1.17 (F7/A0)
- net F7: now also SW8.2
- net F6: now reaches U1.18 (F6/A1)
- net F6: now also SW3.2
- net F5: now reaches U1.19 (F5/A2)
- net F5: now also SW12.A
- net F4: now reaches U1.20 (F4/A3)
- net F4: now also SW12.B
- net D4: now reaches U1.7 (4/D4)
- net D4: now also SW9.2
- net C6: now reaches U1.8 (5/C6)
- net C6: now also SW6.2
- net D7: now reaches U1.9 (6/D7)
- net D7: now also SW4.2
- no-connect marks 0 -> 4
Changed lines of the file:
@@
 P 2300 1550
 F 0 "SW1" H 2300 1805 50  0000 C CNN
-F 1 "SW_PUSH" H 2300 1714 50  0000 C CNN
-F 2 "Keebio-Parts:MX-Alps-Choc-1U-NoLED" H 2300 1550 50  0001 C CNN
+F 1 "1" H 2300 1714 50  0000 C CNN
+F 2 "MX_Only:MXOnly-1U-NoLED" H 2300 1550 50  0001 C CNN
 F 3 "" H 2300 1550 50  0000 C CNN
 	1    2300 1550
@@
 P 3050 1550
 F 0 "SW4" H 3050 1805 50  0000 C CNN
-F 1 "SW_PUSH" H 3050 1714 50  0000 C CNN
-F 2 "Keebio-Parts:MX-Alps-Choc-1U-NoLED" H 3050 1550 50  0001 C CNN
+F 1 "2" H 3050 1714 50  0000 C CNN
+F 2 "MX_Only:MXOnly-1U-NoLED" H 3050 1550 50  0001 C CNN
 F 3 "" H 3050 1550 50  0000 C CNN
 	1    3050 1550
@@
 P 3800 1550
 F 0 "SW6" H 3800 1805 50  0000 C CNN
-F 1 "SW_PUSH" H 3800 1714 50  0000 C CNN
-F 2 "Keebio-Parts:MX-Alps-Choc-1U-NoLED" H 3800 1550 50  0001 C CNN
+F 1 "3" H 3800 1714 50  0000 C CNN
+F 2 "MX_Only:MXOnly-1U-NoLED" H 3800 1550 50  0001 C CNN
 F 3 "" H 3800 1550 50  0000 C CNN
 	1    3800 1550
@@
 P 4550 1550
 F 0 "SW9" H 4550 1805 50  0000 C CNN
-F 1 "SW_PUSH" H 4550 1714 50  0000 C CNN
-F 2 "Keebio-Parts:MX-Alps-Choc-1U-NoLED" H 4550 1550 50  0001 C CNN
+F 1 "4" H 4550 1714 50  0000 C CNN
+F 2 "MX_Only:MXOnly-1U-NoLED" H 4550 1550 50  0001 C CNN
 F 3 "" H 4550 1550 50  0000 C CNN
 	1    4550 1550
@@
 P 2300 2050
 F 0 "SW2" H 2300 2305 50  0000 C CNN
-F 1 "SW_PUSH" H 2300 2214 50  0000 C CNN
-F 2 "Keebio-Parts:MX-Alps-Choc-1U-NoLED" H 2300 2050 50  0001 C CNN
+F 1 "5" H 2300 2214 50  0000 C CNN
+F 2 "MX_Only:MXOnly-1U-NoLED" H 2300 2050 50  0001 C CNN
 F 3 "" H 2300 2050 50  0000 C CNN
 	1    2300 2050
@@
 P 3050 2050
 F 0 "SW5" H 3050 2305 50  0000 C CNN
-F 1 "SW_PUSH" H 3050 2214 50  0000 C CNN
-F 2 "Keebio-Parts:MX-Alps-Choc-1U-NoLED" H 3050 2050 50  0001 C CNN
+F 1 "6" H 3050 2214 50  0000 C CNN
+F 2 "MX_Only:MXOnly-1U-NoLED" H 3050 2050 50  0001 C CNN
 F 3 "" H 3050 2050 50  0000 C CNN
 	1    3050 2050
@@
 P 3800 2050
 F 0 "SW7" H 3800 2305 50  0000 C CNN
-F 1 "SW_PUSH" H 3800 2214 50  0000 C CNN
-F 2 "Keebio-Parts:MX-Alps-Choc-1U-NoLED" H 3800 2050 50  0001 C CNN
+F 1 "7" H 3800 2214 50  0000 C CNN
+F 2 "MX_Only:MXOnly-1U-NoLED" H 3800 2050 50  0001 C CNN
 F 3 "" H 3800 2050 50  0000 C CNN
 	1    3800 2050
@@
 P 4550 2050
 F 0 "SW10" H 4550 2305 50  0000 C CNN
-F 1 "SW_PUSH" H 4550 2214 50  0000 C CNN
-F 2 "Keebio-Parts:MX-Alps-Choc-1U-NoLED" H 4550 2050 50  0001 C CNN
+F 1 "8" H 4550 2214 50  0000 C CNN
+F 2 "MX_Only:MXOnly-1U-NoLED" H 4550 2050 50  0001 C CNN
 F 3 "" H 4550 2050 50  0000 C CNN
 	1    4550 2050
@@
 P 2300 2550
 F 0 "SW3" H 2300 2805 50  0000 C CNN
-F 1 "SW_PUSH" H 2300 2714 50  0000 C CNN
-F 2 "Keebio-Parts:MX-Alps-Choc-2U" H 2300 2550 50  0001 C CNN
+F 1 "ENTER" H 2300 2714 50  0000 C CNN
+F 2 "MX_Only:MXOnly-2U-ReversedStabilizers-NoLED" H 2300 2550 50  0001 C CNN
 F 3 "" H 2300 2550 50  0000 C CNN
 	1    2300 2550
@@
 P 3800 2550
 F 0 "SW8" H 3800 2805 50  0000 C CNN
-F 1 "SW_PUSH" H 3800 2714 50  0000 C CNN
-F 2 "Keebio-Parts:MX-Alps-Choc-1U-NoLED" H 3800 2550 50  0001 C CNN
+F 1 "9" H 3800 2714 50  0000 C CNN
+F 2 "MX_Only:MXOnly-1U-NoLED" H 3800 2550 50  0001 C CNN
 F 3 "" H 3800 2550 50  0000 C CNN
 	1    3800 2550
@@
 P 4550 2550
 F 0 "SW11" H 4550 2805 50  0000 C CNN
-F 1 "SW_PUSH" H 4550 2714 50  0000 C CNN
-F 2 "Keebio-Parts:MX-Alps-Choc-1U-NoLED" H 4550 2550 50  0001 C CNN
+F 1 "0" H 4550 2714 50  0000 C CNN
+F 2 "MX_Only:MXOnly-1U-NoLED" H 4550 2550 50  0001 C CNN
 F 3 "" H 4550 2550 50  0000 C CNN
 	1    4550 2550
@@
 P 6050 2300
 F 0 "SW12" H 6050 2667 50  0000 C CNN
-F 1 "Rotary_Encoder_Switch" H 6050 2576 50  0000 C CNN
+F 1 "ROTARY" H 6050 2576 50  0000 C CNN
 F 2 "Keebio-Parts:RotaryEncoder_Alps_EC11E-Switch_Vertical_H20mm" H 5900 2460 50  0001 C CNN
 F 3 "~" H 6050 2560 50  0001 C CNN
@@
 	3500 2200 2750 2200
 Wire Wire Line
-	2000 2550 2000 2700
-Wire Wire Line
-	2000 2700 1900 2700
-Wire Wire Line
 	3500 2550 3500 2700
-Wire Wire Line
-	3500 2700 2000 2700
-Connection ~ 2000 2700
 Wire Wire Line
 	4250 2550 4250 2700
@@
 L power:GND #PWR0105
 U 1 1 6000E4D0
-P 6450 2400
-F 0 "#PWR0105" H 6450 2150 50  0001 C CNN
-F 1 "GND" H 6455 2227 50  0000 C CNN
-F 2 "" H 6450 2400 50  0001 C CNN
-F 3 "" H 6450 2400 50  0001 C CNN
-	1    6450 2400
-	1    0    0    -1
-$EndComp
-Wire Wire Line
-	6450 2400 6350 2400
+P 6600 2200
+F 0 "#PWR0105" H 6600 1950 50  0001 C CNN
+F 1 "GND" H 6605 2027 50  0000 C CNN
+F 2 "" H 6600 2200 50  0001 C CNN
+F 3 "" H 6600 2200 50  0001 C CNN
+	1    6600 2200
+	1    0    0    -1
+$EndComp
 $Comp
 L power:GND #PWR0106
@@
 Wire Wire Line
 	10850 1400 10500 1400
+Wire Wire Line
+	1900 2700 2000 2700
+$Comp
+L power:+5V #PWR0108
+U 1 1 6000AEF7
+P 10600 1600
+F 0 "#PWR0108" H 10600 1450 50  0001 C CNN
+F 1 "+5V" H 10615 1773 50  0000 C CNN
+F 2 "" H 10600 1600 50  0001 C CNN
+F 3 "" H 10600 1600 50  0001 C CNN
+	1    10600 1600
+	1    0    0    -1
+$EndComp
+Wire Wire Line
+	10600 1600 10500 1600
+Wire Wire Line
+	2000 2550 2000 2700
+Connection ~ 2000 2700
+Wire Wire Line
+	2000 2700 3500 2700
+Text GLabel 5750 2400 0    50   Input ~ 0
+F4
+Text GLabel 5750 2200 0    50   Input ~ 0
+F5
+Text GLabel 10500 1700 2    50   Input ~ 0
+F4
+Text GLabel 10500 1800 2    50   Input ~ 0
+F5
+Text GLabel 6350 2400 2    50   Input ~ 0
+B6
+Wire Wire Line
+	6350 2200 6600 2200
+Text GLabel 9100 1900 0    50   Input ~ 0
+D4
+Text GLabel 9100 2000 0    50   Input ~ 0
+C6
+Text GLabel 9100 2100 0    50   Input ~ 0
+D7
+Text GLabel 9100 2200 0    50   Input ~ 0
+E6
+Text GLabel 9100 2300 0    50   Input ~ 0
+B4
+Text GLabel 9100 2400 0    50   Input ~ 0
+B5
+Text GLabel 4850 1550 1    50   Input ~ 0
+D4
+Text GLabel 4100 1550 1    50   Input ~ 0
+C6
+Text GLabel 3350 1550 1    50   Input ~ 0
+D7
+Text GLabel 2600 1550 1    50   Input ~ 0
+E6
+Text GLabel 4850 2050 1    50   Input ~ 0
+B4
+Text GLabel 4100 2050 1    50   Input ~ 0
+B5
+Text GLabel 10500 2400 2    50   Input ~ 0
+B6
+Text GLabel 10500 2300 2    50   Input ~ 0
+B2
+Text GLabel 10500 2200 2    50   Input ~ 0
+B3
+Text GLabel 3350 2050 1    50   Input ~ 0
+B2
+Text GLabel 2600 2050 1    50   Input ~ 0
+B3
+Text GLabel 10500 2100 2    50   Input ~ 0
+B1
+Text GLabel 10500 2000 2    50   Input ~ 0
+F7
+Text GLabel 10500 1900 2    50   Input ~ 0
+F6
+Text GLabel 4850 2550 1    50   Input ~ 0
+B1
+Text GLabel 4100 2550 1    50   Input ~ 0
+F7
+Text GLabel 2600 2550 1    50   Input ~ 0
+F6
+NoConn ~ 10500 1500
+NoConn ~ 10500 1300
+NoConn ~ 9100 1300
+NoConn ~ 9100 1400
+$Comp
+L Mechanical:MountingHole H1
+U 1 1 600478D8
+P 9350 3550
+F 0 "H1" H 9450 3596 50  0000 L CNN
+F 1 "MountingHole" H 9450 3505 50  0000 L CNN
+F 2 "kbd:M2_Hole_TH" H 9350 3550 50  0001 C CNN
+F 3 "~" H 9350 3550 50  0001 C CNN
+	1    9350 3550
+	1    0    0    -1
+$EndComp
+$Comp
+L Mechanical:MountingHole H2
+U 1 1 60048550
+P 9350 3750
+F 0 "H2" H 9450 3796 50  0000 L CNN
+F 1 "MountingHole" H 9450 3705 50  0000 L CNN
+F 2 "kbd:M2_Hole_TH" H 9350 3750 50  0001 C CNN
+F 3 "~" H 9350 3750 50  0001 C CNN
+	1    9350 3750
+	1    0    0    -1
+$EndComp
+$Comp
+L Mechanical:MountingHole H3
+U 1 1 60048979
+P 9350 3950
+F 0 "H3" H 9450 3996 50  0000 L CNN
+F 1 "MountingHole" H 9450 3905 50  0000 L CNN
+F 2 "kbd:M2_Hole_TH" H 9350 3950 50  0001 C CNN
+F 3 "~" H 9350 3950 50  0001 C CNN
+	1    9350 3950
+	1    0    0    -1
+$EndComp
+$Comp
+L Mechanical:MountingHole H4
+U 1 1 60048C90
+P 9350 4150
+F 0 "H4" H 9450 4196 50  0000 L CNN
+F 1 "MountingHole" H 9450 4105 50  0000 L CNN
+F 2 "kbd:M2_Hole_TH" H 9350 4150 50  0001 C CNN
+F 3 "~" H 9350 4150 50  0001 C CNN
+	1    9350 4150
+	1    0    0    -1
+$EndComp
 $EndSCHEMATC
